File: EGB240_Transistor_75x50mm.brd (EAGLE design)
At the start: 49.6 x 44.9 mm, 12 parts, among them Q1 2N4126, U1 74HC14

Commit message: Added Gerber files
Parts:
- Q1: value 2N4126 -> PN200
- X1: value (none) -> PS1720P02
Connections:
- new net N$9: U1.P$4, X1.P$1
- net GND: no longer U1.P$3
- net N$7: now also U1.P$3; no longer X1.P$1
Routing:
- net N$7: track 53.1 -> 17.9 mm
- net N$9: track 0.00 -> 22.9 mm
- net GND: track 104.2 -> 116.1 mm
Other:
- board size 49.6 x 44.9 mm -> 45.8 x 43.6 mm
Changed lines of the file:
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@@
 <board>
 <plain>
-<wire x1="0" y1="0" x2="49.6" y2="0" width="0" layer="20"/>
-<wire x1="49.6" y1="0" x2="49.6" y2="44.92" width="0" layer="20"/>
-<wire x1="49.6" y1="44.92" x2="0" y2="44.92" width="0" layer="20"/>
-<wire x1="0" y1="44.92" x2="0" y2="0" width="0" layer="20"/>
-<text x="4.08" y="40.11" size="1.27" layer="21" font="vector" ratio="12" rot="SR0">EGB240 n8802530
+<wire x1="0" y1="0" x2="45.79" y2="0" width="0" layer="20"/>
+<wire x1="45.79" y1="0" x2="45.79" y2="43.65" width="0" layer="20"/>
+<wire x1="45.79" y1="43.65" x2="0" y2="43.65" width="0" layer="20"/>
+<wire x1="0" y1="43.65" x2="0" y2="0" width="0" layer="20"/>
+<text x="21.86" y="2.01" size="1.27" layer="21" font="vector" ratio="12" rot="SR0">EGB240 n8802530
 Nathan Ramage</text>
-<wire x1="1" y1="1" x2="1" y2="43.92" width="0.4064" layer="21"/>
-<wire x1="1" y1="43.92" x2="48.6" y2="43.92" width="0.4064" layer="21"/>
-<wire x1="48.6" y1="43.92" x2="48.6" y2="1" width="0.4064" layer="21"/>
-<wire x1="48.6" y1="1" x2="1" y2="1" width="0.4064" layer="21"/>
-<wire x1="0" y1="44.92" x2="0" y2="0" width="2" layer="40"/>
-<wire x1="0" y1="0" x2="49.6" y2="0" width="2" layer="40"/>
-<wire x1="49.6" y1="0" x2="49.6" y2="44.92" width="2" layer="40"/>
-<wire x1="49.6" y1="44.92" x2="0" y2="44.92" width="2" layer="40"/>
+<wire x1="1" y1="1" x2="1" y2="42.65" width="0.4064" layer="21"/>
+<wire x1="44.79" y1="42.65" x2="44.79" y2="1" width="0.4064" layer="21"/>
+<wire x1="44.79" y1="1" x2="1" y2="1" width="0.4064" layer="21"/>
+<wire x1="0" y1="43.65" x2="0" y2="0" width="2" layer="40"/>
+<wire x1="0" y1="0" x2="45.79" y2="0" width="2" layer="40"/>
+<wire x1="45.79" y1="0" x2="45.79" y2="43.65" width="2" layer="40"/>
+<wire x1="45.79" y1="43.65" x2="0" y2="43.65" width="2" layer="40"/>
 </plain>
 <attributes>
@@
 <element name="R1" library="EGB240" package="AXIAL-P2.54" value="22k" x="19.05" y="13.97" rot="R180"/>
 <element name="R2" library="EGB240" package="AXIAL-P2.54" value="15k" x="8.89" y="11.43"/>
-<element name="C1" library="EGB240" package="CAP-DISC-P5.08" value="15n" x="8.89" y="5.08"/>
+<element name="C1" library="EGB240" package="CAP-DISC-P5.08" value="15n" x="8.89" y="5.08" smashed="yes">
+<attribute name="NAME" x="8.89" y="1.524" size="1.27" layer="21" align="bottom-center"/>
+</element>
 <element name="J1" library="EGB240" package="BATT-3V" value="" x="20.32" y="34.29"/>
 <element name="S1" library="EGB240" package="SS-12" value="" x="10.16" y="36.83" rot="R90"/>
-<element name="X1" library="EGB240" package="PS1720P02" value="" x="34.29" y="27.94" rot="R90"/>
+<element name="X1" library="EGB240" package="PS1720P02" value="PS1720P02" x="34.29" y="27.94" rot="R90"/>
 <element name="C2" library="EGB240" package="CAP-RB-P2.0-D5.0" value="33u" x="29.21" y="16.51"/>
-<element name="R3" library="EGB240" package="AXIAL-P2.54" value="27k" x="8.89" y="8.89"/>
+<element name="R3" library="EGB240" package="AXIAL-P2.54" value="27k" x="8.89" y="8.89" smashed="yes">
+<attribute name="NAME" x="5.08" y="7.874" size="1.27" layer="21" align="bottom-center"/>
+</element>
 <element name="D1" library="EGB240" package="DO35-P2.54" value="" x="24.13" y="13.97"/>
 <element name="R4" library="EGB240" package="AXIAL-P10.16" value="15k" x="26.67" y="7.62"/>
-<element name="Q1" library="transistor-pnp" package="TO92-CBE" value="2N4126" x="17.78" y="7.62" rot="MR270"/>
+<element name="Q1" library="transistor-pnp" package="TO92-CBE" value="PN200" x="17.78" y="7.62" smashed="yes" rot="MR270">
+<attribute name="NAME" x="13.462" y="10.16" size="1.27" layer="25" ratio="10" rot="R270"/>
+<attribute name="VALUE" x="13.97" y="3.048" size="1.27" layer="27" ratio="10"/>
+</element>
 </elements>
 <signals>
@@
 <contactref element="C2" pad="P$2"/>
 <contactref element="C1" pad="P$2"/>
-<contactref element="X1" pad="P$2"/>
 <contactref element="J1" pad="P$2"/>
-<contactref element="U1" pad="P$3"/>
 <contactref element="U1" pad="P$9"/>
 <contactref element="U1" pad="P$11"/>
 <contactref element="U1" pad="P$13"/>
 <wire x1="20.32" y1="29.21" x2="21.59" y2="34.29" width="1.016" layer="16"/>
-<wire x1="10.16" y1="29.21" x2="11.728825" y2="22.93470625" width="1.016" layer="16"/>
-<wire x1="11.728825" y1="22.93470625" x2="12.7" y2="19.05" width="1.016" layer="16"/>
-<wire x1="12.7" y1="19.05" x2="15.24" y2="29.21" width="1.016" layer="16"/>
-<wire x1="15.24" y1="29.21" x2="15.24" y2="26.67" width="1.016" layer="16"/>
-<wire x1="15.24" y1="26.67" x2="20.32" y2="26.67" width="1.016" layer="16"/>
-<wire x1="20.32" y1="26.67" x2="20.32" y2="29.21" width="1.016" layer="16"/>
 <wire x1="30.21" y1="16.51" x2="30.21" y2="18.05" width="1.016" layer="16"/>
 <wire x1="30.21" y1="18.05" x2="29.21" y2="19.05" width="1.016" layer="16"/>
 <wire x1="29.21" y1="19.05" x2="22.86" y2="19.05" width="1.016" layer="16"/>
-<wire x1="11.43" y1="5.08" x2="5.08" y2="2.54" width="1.016" layer="16"/>
-<wire x1="5.08" y1="2.54" x2="3.81" y2="6.35" width="1.016" layer="16"/>
-<wire x1="3.81" y1="6.35" x2="3.81" y2="22.86" width="1.016" layer="16"/>
-<wire x1="3.81" y1="22.86" x2="11.728825" y2="22.93470625" width="1.016" layer="16"/>
-<wire x1="22.86" y1="19.05" x2="20.32" y2="29.21" width="1.016" layer="16"/>
-<wire x1="34.29" y1="32.94" x2="21.59" y2="34.29" width="1.016" layer="16"/>
+<contactref element="X1" pad="P$2"/>
+<wire x1="20.32" y1="29.21" x2="20.32" y2="25.4" width="1.016" layer="16"/>
+<wire x1="20.32" y1="25.4" x2="15.24" y2="25.4" width="1.016" layer="16"/>
+<wire x1="15.24" y1="25.4" x2="15.24" y2="29.21" width="1.016" layer="16"/>
+<wire x1="20.32" y1="25.4" x2="36.83" y2="25.4" width="1.016" layer="16"/>
+<wire x1="36.83" y1="25.4" x2="36.83" y2="16.51" width="1.016" layer="16"/>
+<wire x1="36.83" y1="16.51" x2="30.21" y2="16.51" width="1.016" layer="16"/>
+<wire x1="36.83" y1="25.4" x2="36.83" y2="30.4" width="1.016" layer="16"/>
+<wire x1="36.83" y1="30.4" x2="34.29" y2="32.94" width="1.016" layer="16" curve="90"/>
+<wire x1="15.24" y1="25.4" x2="10.16" y2="25.4" width="1.016" layer="16"/>
+<wire x1="10.16" y1="25.4" x2="10.16" y2="29.21" width="1.016" layer="16"/>
+<wire x1="11.43" y1="5.08" x2="11.43" y2="2.54" width="1.016" layer="16"/>
+<wire x1="11.43" y1="2.54" x2="3.81" y2="2.54" width="1.016" layer="16"/>
+<wire x1="3.81" y1="2.54" x2="3.81" y2="25.4" width="1.016" layer="16"/>
+<wire x1="3.81" y1="25.4" x2="10.16" y2="25.4" width="1.016" layer="16"/>
 </signal>
 <signal name="N$1">
@@
 <wire x1="5.08" y1="6.35" x2="6.35" y2="5.08" width="1.016" layer="16"/>
 </signal>
-<signal name="N$7">
-<contactref element="R2" pad="P$2"/>
-<contactref element="X1" pad="P$1"/>
-<contactref element="Q1" pad="E"/>
-<contactref element="U1" pad="P$2"/>
-<wire x1="17.78" y1="10.16" x2="10.16" y2="11.43" width="1.016" layer="16"/>
-<wire x1="10.16" y1="11.43" x2="10.16" y2="19.05" width="1.016" layer="16"/>
-<wire x1="34.29" y1="22.94" x2="34.29" y2="10.16" width="1.016" layer="16"/>
-<wire x1="34.29" y1="10.16" x2="35.56" y2="8.89" width="1.016" layer="16"/>
-<wire x1="35.56" y1="8.89" x2="35.56" y2="6.35" width="1.016" layer="16"/>
-<wire x1="35.56" y1="6.35" x2="34.29" y2="5.08" width="1.016" layer="16"/>
-<wire x1="34.29" y1="5.08" x2="31.75" y2="3.81" width="1.016" layer="16"/>
-<wire x1="31.75" y1="3.81" x2="22.86" y2="10.16" width="1.016" layer="16"/>
-<wire x1="22.86" y1="10.16" x2="17.78" y2="10.16" width="1.016" layer="16"/>
-</signal>
 <signal name="N$8">
 <contactref element="J1" pad="P$1"/>
@@
 <wire x1="7.62" y1="33.02" x2="7.62" y2="29.21" width="1.016" layer="16"/>
 </signal>
+<signal name="N$9">
+<contactref element="X1" pad="P$1"/>
+<contactref element="U1" pad="P$4"/>
+<wire x1="15.24" y1="19.05" x2="15.24" y2="22.86" width="1.016" layer="16"/>
+<wire x1="15.24" y1="22.86" x2="34.21" y2="22.86" width="1.016" layer="16"/>
+<wire x1="34.21" y1="22.86" x2="34.29" y2="22.94" width="1.016" layer="16"/>
+</signal>
+<signal name="N$7">
+<contactref element="U1" pad="P$3"/>
+<contactref element="U1" pad="P$2"/>
+<contactref element="Q1" pad="E"/>
+<contactref element="R2" pad="P$2"/>
+<wire x1="17.78" y1="10.16" x2="10.16" y2="11.43" width="1.016" layer="16"/>
+<wire x1="10.16" y1="11.43" x2="10.16" y2="19.05" width="1.016" layer="16"/>
+<wire x1="10.16" y1="19.05" x2="12.7" y2="19.05" width="1.016" layer="16"/>
+</signal>
 </signals>
